File: ergogen-kikad/design/alternatives/five-column-15u/pcbs/macropad.kicad_pcb (KiCad board)
At the start: 2 copper layers, 98 x 96 mm, 23 parts, among them J1 JST-PH S2B-PH-K-S

Commit message: Revise selected 1.5U layout with aligned caps and central battery
Parts:
- BAT1: value 301230 110mAh max 32x13x3.5 z=-1.4 -> 301055 220mAh max 57.5x10.5x3.5 z=-1.4; footprint Protected_301230_Battery_Envelope -> Protected_301055_Battery_Envelope
- WELL1: value Battery well 32.6x13.6 -> Battery well 58.1x11.1
- moved PWR1 56.3 mm to (91.5, -53.0)
- moved J1 51.5 mm to (89.5, -43.0)
- moved RST1 41.5 mm to (81.5, -53.0)
- moved BAT1 39.8 mm to (32.0, -48.0)
- moved WELL1 39.8 mm to (32.0, -48.0)
- moved LCD1 36.9 mm to (60.0, -85.8), turned to 0 degrees
- moved S10 5.00 mm to (87.1, -29.2)
- moved S9 5.00 mm to (87.1, -66.8)
Changed lines of the file:
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@@
     )
     (module PG1350_1U (layer F.Cu)
-      (at 87.10000000000001 -61.75 0)
+      (at 87.10000000000001 -66.75 0)
       (fp_text reference "S9" (at 0 0) (layer F.SilkS) hide
         (effects (font (size 1 1) (thickness 0.15))))
@@
     )
     (module PG1350_1U (layer F.Cu)
-      (at 87.10000000000001 -34.25 0)
+      (at 87.10000000000001 -29.25 0)
       (fp_text reference "S10" (at 0 0) (layer F.SilkS) hide
         (effects (font (size 1 1) (thickness 0.15))))
@@
     )
 (module Nice_View_Socketed_Module (layer F.Cu)
-      (at 23.1 -85.75 180)
+      (at 60 -85.75 0)
       (fp_text reference "LCD1" (at -16.7 0) (layer F.Fab) hide (effects (font (size 1 1) (thickness 0.15))))
       (fp_text value "nice!view" (at 0 0) (layer F.Fab) hide (effects (font (size 1 1) (thickness 0.15))))
@@
     )
 (module JST_PH_S2B_PH_K_Horizontal (layer F.Cu)
-    (at 50 -10 -90)
+    (at 89.5 -43 -90)
     (fp_text reference "J1" (at 0 0) (layer F.Fab) hide (effects (font (size 1 1) (thickness 0.15))))
     (fp_text value "JST-PH S2B-PH-K-S" (at 0 0) (layer F.Fab) hide (effects (font (size 1 1) (thickness 0.15))))
@@
   )
 (module CK_OS102011MS2QN1 (layer F.Cu)
-    (at 50 -91 0)
+    (at 91.5 -53 0)
     (fp_text reference "PWR1" (at 0 0) (layer F.Fab) hide (effects (font (size 1 1) (thickness 0.15))))
     (fp_text value "OS102011MS2QN1" (at 0 0) (layer F.Fab) hide (effects (font (size 1 1) (thickness 0.15))))
@@
   )
 (module SW_PUSH_6mm_H4_3mm (layer F.Cu)
-    (at 50 -80 0)
+    (at 81.5 -53 0)
     (fp_text reference "RST1" (at 0 0) (layer F.Fab) hide (effects (font (size 1 1) (thickness 0.15))))
     (fp_text value "6mm top-actuated tactile" (at 0 0) (layer F.Fab) hide (effects (font (size 1 1) (thickness 0.15))))
@@
     (pad 2 thru_hole circle (at 3.25 2.25) (size 2 2) (drill 1.1) (layers *.Cu *.Mask) (net 1 "GND"))
   )
-(module Protected_301230_Battery_Envelope (layer F.Cu)
-    (at 20 -10 0)
+(module Protected_301055_Battery_Envelope (layer F.Cu)
+    (at 32 -48 0)
     (fp_text reference "BAT1" (at 0 0) (layer F.Fab) hide (effects (font (size 1 1) (thickness 0.15))))
-    (fp_text value "301230 110mAh max 32x13x3.5 z=-1.4" (at 0 0) (layer F.Fab) hide (effects (font (size 1 1) (thickness 0.15))))
-    (fp_text user "301230 110mAh" (at 0 -1) (layer Cmts.User) (effects (font (size 1.2 1.2) (thickness 0.15))))
-    (fp_text user "32 x 13 x 3.5 MAX" (at 0 1.5) (layer Cmts.User) (effects (font (size 0.9 0.9) (thickness 0.13))))
-    (fp_line (start -16 -6.5) (end 16 -6.5) (layer Cmts.User) (width 0.12))
-    (fp_line (start 16 -6.5) (end 16 6.5) (layer Cmts.User) (width 0.12))
-    (fp_line (start 16 6.5) (end -16 6.5) (layer Cmts.User) (width 0.12))
-    (fp_line (start -16 6.5) (end -16 -6.5) (layer Cmts.User) (width 0.12))
+    (fp_text value "301055 220mAh max 57.5x10.5x3.5 z=-1.4" (at 0 0) (layer F.Fab) hide (effects (font (size 1 1) (thickness 0.15))))
+    (fp_text user "301055 220mAh" (at 0 -1) (layer Cmts.User) (effects (font (size 1.2 1.2) (thickness 0.15))))
+    (fp_text user "57.5 x 10.5 x 3.5 MAX" (at 0 1.5) (layer Cmts.User) (effects (font (size 0.9 0.9) (thickness 0.13))))
+    (fp_line (start -28.75 -5.25) (end 28.75 -5.25) (layer Cmts.User) (width 0.12))
+    (fp_line (start 28.75 -5.25) (end 28.75 5.25) (layer Cmts.User) (width 0.12))
+    (fp_line (start 28.75 5.25) (end -28.75 5.25) (layer Cmts.User) (width 0.12))
+    (fp_line (start -28.75 5.25) (end -28.75 -5.25) (layer Cmts.User) (width 0.12))
   )
 (module Battery_Well (layer F.Cu)
-      (at 20 -10 0)
+      (at 32 -48 0)
       (fp_text reference "WELL1" (at 0 0) (layer F.Fab) hide (effects (font (size 1 1) (thickness 0.15))))
-      (fp_text value "Battery well 32.6x13.6" (at 0 0) (layer F.Fab) hide (effects (font (size 1 1) (thickness 0.15))))
-      (fp_line (start -15.8 -6.8) (end 15.8 -6.8) (layer Edge.Cuts) (width 0.05))
-(fp_line (start 15.8 -6.8) (end 16.3 -6.3) (layer Edge.Cuts) (width 0.05))
-(fp_line (start 16.3 -6.3) (end 16.3 6.3) (layer Edge.Cuts) (width 0.05))
-(fp_line (start 16.3 6.3) (end 15.8 6.8) (layer Edge.Cuts) (width 0.05))
-(fp_line (start 15.8 6.8) (end -15.8 6.8) (layer Edge.Cuts) (width 0.05))
-(fp_line (start -15.8 6.8) (end -16.3 6.3) (layer Edge.Cuts) (width 0.05))
-(fp_line (start -16.3 6.3) (end -16.3 -6.3) (layer Edge.Cuts) (width 0.05))
-(fp_line (start -16.3 -6.3) (end -15.8 -6.8) (layer Edge.Cuts) (width 0.05))
+      (fp_text value "Battery well 58.1x11.1" (at 0 0) (layer F.Fab) hide (effects (font (size 1 1) (thickness 0.15))))
+      (fp_line (start -28.55 -5.55) (end 28.55 -5.55) (layer Edge.Cuts) (width 0.05))
+(fp_line (start 28.55 -5.55) (end 29.05 -5.05) (layer Edge.Cuts) (width 0.05))
+(fp_line (start 29.05 -5.05) (end 29.05 5.05) (layer Edge.Cuts) (width 0.05))
+(fp_line (start 29.05 5.05) (end 28.55 5.55) (layer Edge.Cuts) (width 0.05))
+(fp_line (start 28.55 5.55) (end -28.55 5.55) (layer Edge.Cuts) (width 0.05))
+(fp_line (start -28.55 5.55) (end -29.05 5.05) (layer Edge.Cuts) (width 0.05))
+(fp_line (start -29.05 5.05) (end -29.05 -5.05) (layer Edge.Cuts) (width 0.05))
+(fp_line (start -29.05 -5.05) (end -28.55 -5.55) (layer Edge.Cuts) (width 0.05))
     )
   (gr_line (start 1.5 0) (end 96.5 0) (angle 90) (layer Edge.Cuts) (width 0.15))
